File: _autosave-keeboard.kicad_sch (KiCad schematic)
At the start: 179 parts, among them SW1 SW_Push, SW10 SW_Push, SW11 SW_Push, SW12 SW_Push, SW13 SW_Push, SW14 SW_Push, SW15 SW_Push, SW16 SW_Push, SW17 SW_Push, SW18 SW_Push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

Commit message: started pcb
Parts:
- renumbered D15 to D10, D16 to D11, D17 to D12, D18 to D13, D19 to D14, D20 to D15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
