File: keeboard.kicad_pcb (KiCad board)
At the start: 2 copper layers, 309 x 121 mm, 179 parts, among them SW1 SW_Push, SW10 SW_Push, SW11 SW_Push, SW12 SW_Push, SW13 SW_Push, SW14 SW_Push, SW15 SW_Push, SW16 SW_Push, SW17 SW_Push, SW18 SW_Push, SW19 SW_Push, SW2 SW_Push, SW20 SW_Push, SW21 SW_Push, SW22 SW_Push, SW23 SW_Push, SW24 SW_Push, SW25 SW_Push, SW26 SW_Push, SW27 SW_Push, SW28 SW_Push, SW29 SW_Push, SW3 SW_Push, SW30 SW_Push, SW31 SW_Push, SW32 SW_Push, SW33 SW_Push, SW34 SW_Push, SW35 SW_Push, SW36 SW_Push, SW37 SW_Push, SW38 SW_Push, SW39 SW_Push, SW4 SW_Push, SW40 SW_Push, SW41 SW_Push, SW42 SW_Push, SW43 SW_Push, SW44 SW_Push, SW45 SW_Push, SW46 SW_Push, SW47 SW_Push, SW48 SW_Push, SW49 SW_Push, SW5 SW_Push, SW50 SW_Push, SW51 SW_Push, SW52 SW_Push, SW53 SW_Push, SW54 SW_Push, SW55 SW_Push, SW56 SW_Push, SW57 SW_Push, SW58 SW_Push, SW59 SW_Push, SW6 SW_Push, SW60 SW_Push, SW61 SW_Push, SW63 SW_Push, SW64 SW_Push, SW65 SW_Push, SW66 SW_Push, SW67 SW_Push, SW68 SW_Push, SW69 SW_Push, SW7 SW_Push, SW70 SW_Push, SW71 SW_Push, SW72 SW_Push, SW73 SW_Push, SW74 SW_Push, SW75 SW_Push, SW76 SW_Push, SW77 SW_Push, SW78 SW_Push, SW79 SW_Push, SW8 SW_Push, SW82 SW_Push, SW83 SW_Push, SW84 SW_Push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

Commit message: e
Parts:
- removed D85, D86, D87: 1N4148, Diode_THT:D_DO-35_SOD27_P7.62mm_Horizontal
- removed H6: MountingHole, MountingHole:MountingHole_2.2mm_M2
- removed SW85, SW86, SW87: SW_Push, PCM_marbastlib-mx:SW_MX_1u
- added D62: 1N4148, Diode_THT:D_DO-35_SOD27_P7.62mm_Horizontal, B.Cu at (101.7, 174.6)
- added D80: 1N4148, Diode_THT:D_DO-35_SOD27_P7.62mm_Horizontal, B.Cu at (268.4, 193.6)
- added D81: 1N4148, Diode_THT:D_DO-35_SOD27_P7.62mm_Horizontal, B.Cu at (287.4, 193.6)
- added SW62: SW_Push, PCM_marbastlib-mx:SW_MX_1u, F.Cu at (96.6, 170.6)
- added SW80: SW_Push, PCM_marbastlib-mx:SW_MX_1u, F.Cu at (263.3, 189.6)
- added SW81: SW_Push, PCM_marbastlib-mx:SW_MX_1u, F.Cu at (282.4, 189.6)
- D1, D10, D11, D12, D13, D14, D15, D16, D17, D18, D19, D2, D20, D21, D22, D23, D24, D25, D26, D27, D28, D29, D3, D30, D31, D32, D33, D34, D35, D36, D37, D38, D39, D4, D40, D41, D42, D43, D44, D45, D46, D47, D48, D49, D5, D50, D51, D52, D53, D54, D55, D56, D57, D58, D59, D6, D60, D61, D63, D64, D65, D66, D67, D68, D69, D7, D70, D71, D72, D73, D74, D75, D76, D77, D78, D79, D8, D82, D83, D84, D9: moved to B.Cu
- S2: footprint PCM_marbastlib-mx:STAB_MX_2.25u -> PCM_marbastlib-mx:STAB_MX_P_6.25u
- S3: footprint PCM_marbastlib-mx:STAB_MX_P_6.25u -> PCM_marbastlib-mx:STAB_MX_2.25u
- moved A1 344.9 mm to (357.2, 81.8)
- moved SW16 247.6 mm to (339.5, 94.3)
- moved SW31 234.7 mm to (339.5, 113.4)
- moved SW15 229.5 mm to (320.4, 94.3)
- moved SW46 222.0 mm to (339.5, 132.4)
- moved SW14 212.8 mm to (301.4, 94.3)
- moved SW45 207.8 mm to (315.7, 132.4)
- moved SW30 204.6 mm to (310.9, 113.4)
- moved SW60 198.3 mm to (339.5, 151.5)
- moved SW13 197.6 mm to (282.4, 94.3)
- moved SW84 196.8 mm to (339.5, 189.6)
- moved SW83 192.0 mm to (320.4, 189.6)
- moved D75 191.3 mm to (61.2, 193.6), turned to 90 degrees
- moved SW82 190.3 mm to (301.4, 189.6)
- moved SW11 186.3 mm to (244.2, 94.3)
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Connections:
- A1 pad 13: Net-(A1-GND-Pad13) -> unconnected-(A1-GND-Pad13)_4
- A1 pad 18: Net-(A1-GND-Pad13) -> unconnected-(A1-GND-Pad13)_2
- A1 pad 23: Net-(A1-GND-Pad13) -> unconnected-(A1-GND-Pad13)_3
- A1 pad 28: Net-(A1-GND-Pad13) -> unconnected-(A1-GND-Pad13)_6
- A1 pad 3: Net-(A1-GND-Pad13) -> unconnected-(A1-GND-Pad13)
- A1 pad 38: Net-(A1-GND-Pad13) -> unconnected-(A1-GND-Pad13)_1
- A1 pad 8: Net-(A1-GND-Pad13) -> unconnected-(A1-GND-Pad13)_5
- D17 pad 1: /ROW1 -> /ROW2
- D18 pad 1: /ROW1 -> /ROW2
- D19 pad 1: /ROW1 -> /ROW2
- D2 pad 1: /ROW2 -> /ROW1
- D20 pad 1: /ROW1 -> /ROW2
- D21 pad 1: /ROW1 -> /ROW2
- D3 pad 1: /ROW3 -> /ROW1
- D32 pad 1: /ROW2 -> /ROW3
- D33 pad 1: /ROW2 -> /ROW3
- D34 pad 1: /ROW2 -> /ROW3
- D35 pad 1: /ROW2 -> /ROW3
- D4 pad 1: /ROW4 -> /ROW1
- D47 pad 1: /ROW3 -> /ROW4
- D48 pad 1: /ROW3 -> /ROW4
- D49 pad 1: /ROW3 -> /ROW4
- D5 pad 1: /ROW5 -> /ROW1
- D6 pad 1: /ROW6 -> /ROW1
- D61 pad 1: /ROW4 -> /ROW5
- D63 pad 1: /ROW4 -> /ROW5
- D76 pad 1: /ROW5 -> /ROW6
- D77 pad 1: /ROW5 -> /ROW6
- SW10 pad 1: /COL5 -> /COL10
- SW11 pad 1: /COL6 -> /COL11
- SW12 pad 1: /COL7 -> /COL12
- SW13 pad 1: /COL8 -> /COL13
- SW14 pad 1: /COL9 -> /COL14
- SW15 pad 1: /COL10 -> /COL15
- SW16 pad 1: /COL11 -> /COL16
- SW17 pad 1: /COL12 -> /COL1
- SW18 pad 1: /COL13 -> /COL2
- SW19 pad 1: /COL14 -> /COL3
- SW2 pad 1: /COL1 -> /COL2
- SW20 pad 1: /COL15 -> /COL4
- SW21 pad 1: /COL16 -> /COL5
- SW22 pad 1: /COL2 -> /COL6
- SW23 pad 1: /COL3 -> /COL7
- SW24 pad 1: /COL4 -> /COL8
- SW25 pad 1: /COL5 -> /COL9
- SW26 pad 1: /COL6 -> /COL10
- SW27 pad 1: /COL7 -> /COL11
- SW28 pad 1: /COL8 -> /COL12
- SW29 pad 1: /COL9 -> /COL13
- SW3 pad 1: /COL1 -> /COL3
- SW30 pad 1: /COL10 -> /COL14
- SW31 pad 1: /COL11 -> /COL16
- SW32 pad 1: /COL12 -> /COL1
- SW33 pad 1: /COL13 -> /COL2
- SW34 pad 1: /COL14 -> /COL3
- SW35 pad 1: /COL16 -> /COL4
- SW36 pad 1: /COL2 -> /COL5
- SW37 pad 1: /COL3 -> /COL6
- SW38 pad 1: /COL4 -> /COL7
- SW39 pad 1: /COL5 -> /COL8
- SW4 pad 1: /COL1 -> /COL4
- SW40 pad 1: /COL6 -> /COL9
- SW41 pad 1: /COL7 -> /COL10
- SW42 pad 1: /COL8 -> /COL11
- SW43 pad 1: /COL9 -> /COL12
- SW44 pad 1: /COL10 -> /COL13
- SW45 pad 1: /COL11 -> /COL14
- SW46 pad 1: /COL12 -> /COL16
- SW47 pad 1: /COL13 -> /COL1
- SW48 pad 1: /COL14 -> /COL2
- SW49 pad 1: /COL16 -> /COL3
- SW5 pad 1: /COL1 -> /COL5
- SW50 pad 1: /COL2 -> /COL4
- SW51 pad 1: /COL3 -> /COL5
- SW52 pad 1: /COL4 -> /COL6
- SW53 pad 1: /COL5 -> /COL7
- SW54 pad 1: /COL6 -> /COL8
- SW55 pad 1: /COL7 -> /COL9
- SW56 pad 1: /COL8 -> /COL10
- SW57 pad 1: /COL9 -> /COL11
- SW58 pad 1: /COL10 -> /COL12
- SW59 pad 1: /COL11 -> /COL13
- SW6 pad 1: /COL1 -> /COL6
- SW60 pad 1: /COL12 -> /COL16
- SW61 pad 1: /COL13 -> /COL1
- SW63 pad 1: /COL16 -> /COL4
- SW64 pad 1: /COL3 -> /COL5
- SW65 pad 1: /COL4 -> /COL6
- SW66 pad 1: /COL5 -> /COL7
- SW67 pad 1: /COL6 -> /COL8
- SW68 pad 1: /COL7 -> /COL9
- SW69 pad 1: /COL8 -> /COL10
- SW7 pad 1: /COL2 -> /COL7
- SW70 pad 1: /COL9 -> /COL11
- SW71 pad 1: /COL10 -> /COL12
- SW72 pad 1: /COL11 -> /COL13
- SW73 pad 1: /COL12 -> /COL15
- SW74 pad 1: /COL13 -> /COL16
- SW75 pad 1: /COL2 -> /COL1
- SW76 pad 1: /COL15 -> /COL2
- SW77 pad 1: /COL16 -> /COL3
- SW78 pad 1: /COL3 -> /COL8
- SW79 pad 1: /COL8 -> /COL11
- SW8 pad 1: /COL3 -> /COL8
- SW82 pad 1: /COL11 -> /COL14
- SW83 pad 1: /COL12 -> /COL15
- SW84 pad 1: /COL13 -> /COL16
- SW9 pad 1: /COL4 -> /COL9
Routing:
- net /COL1: track 0.00 -> 415.7 mm
- net /COL2: track 0.00 -> 396.2 mm
- net /ROW6: track 0.00 -> 385.2 mm
- net /COL3: track 0.00 -> 382.1 mm
- net /ROW5: track 0.00 -> 359.2 mm
- net /ROW4: track 0.00 -> 347.4 mm
- net /COL4: track 0.00 -> 345.2 mm
- net /ROW3: track 0.00 -> 333.3 mm
- net /ROW2: track 0.00 -> 324.1 mm
- net /COL5: track 0.00 -> 323.5 mm
- net /ROW1: track 0.00 -> 307.6 mm
- net /COL6: track 0.00 -> 294.4 mm
- net /COL8: track 0.00 -> 280.7 mm
- net /COL7: track 0.00 -> 274.6 mm
- net /COL11: track 0.00 -> 236.1 mm
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- added copper zone on B.Cu, net (none)
- added copper zone on F.Cu, net (none)
Other:
- board size 309 x 121 mm -> 342.5 x 122.6 mm
